File: ublox-breakout.kicad_sch (KiCad schematic)
At the start: 30 parts, among them J1 Conn_Coaxial, J2 Conn_01x07, J3 Conn_01x07, U1 AT2659S, U2 SAFFB1G56KB0F0A, U3 UBX-G7020-KT, X1 26MHz, Y1 32.768k

Commit message: Finish layout
Parts:
- removed J2, J3: Conn_01x07, Connector_PinHeader_2.54mm:PinHeader_1x07_P2.54mm_Vertical, symbol Connector_Generic:Conn_01x07
- added H1, H2: ToolingHole, ToolingHole:ToolingHole_JLCSMT, symbol Mechanical:MountingHole
- added J2, J3: Conn_01x08, Connector_PinHeader_2.54mm:PinHeader_1x08_P2.54mm_Vertical, symbol Connector_Generic:Conn_01x08
Connections:
- net +3V3: now also J2.1 (Pin_1)
- net +BATT: now also J2.3 (Pin_3)
- net GND: now also J2.2 (Pin_2), J3.7 (Pin_7)
- net PIO0: now also J2.4 (Pin_4)
- net PIO1: now also J2.5 (Pin_5)
- net PIO13: now also J2.6 (Pin_6)
- net PIO14: now also J2.7 (Pin_7)
- net PIO15: now also J2.8 (Pin_8)
- net RX: now also J3.2 (Pin_2)
- net SCL: now also J3.3 (Pin_3)
- net SDA: now also J3.4 (Pin_4)
- net TIME1: now also J3.6 (Pin_6)
- net TIME2: now also J3.8 (Pin_8)
- net TX: now also J3.1 (Pin_1)
- net ~{SPI_EN}: now also J3.5 (Pin_5)
